Commit message: implemented neural network and linked motor neurons to synapses

File: body.urdf (robot description, URDF)
Before this commit: robot robot, 3 links, 2 joints
Joints:
- removed joint Torso_Back_Leg
- removed joint Torso_Front_Leg
- added joint Torso_BackLeg: type revolute, parent Torso, child Back_Leg, origin xyz=-0.5 0 1 rpy=0 0 0, axis 0 1 0, limit lower=-3.14159 upper=3.14159 effort=0.0 velocity=0.0
- added joint Torso_FrontLeg: type revolute, parent Torso, child Front_Leg, origin xyz=0.5 0 1 rpy=0 0 0, axis 0 1 0, limit lower=-3.14159 upper=3.14159 effort=0.0 velocity=0.0

Commit message: converted structure of bot and NN into a quadrupedal walker, can run parallel hill climber with new bot structure

File: body.urdf (robot description, URDF)
Before this commit: robot robot, 3 links, 2 joints
Links:
- added link Back_Leg_Lower, mass 1; collision box size=0.2 0.2 1; visual box size=0.2 0.2 1
- added link Front_Leg_Lower, mass 1; collision box size=0.2 0.2 1; visual box size=0.2 0.2 1
- added link Left_Leg, mass 1; collision box size=1 0.2 0.2; visual box size=1 0.2 0.2
- added link Left_Leg_Lower, mass 1; collision box size=0.2 0.2 1; visual box size=0.2 0.2 1
- added link Right_Leg, mass 1; collision box size=1 0.2 0.2; visual box size=1 0.2 0.2
- added link Right_Leg_Lower, mass 1; collision box size=0.2 0.2 1; visual box size=0.2 0.2 1
- link Back_Leg: geometry collision box size=0.2 1 0.2; visual box size=0.2 1 0.2
- link Front_Leg: geometry collision box size=0.2 1 0.2; visual box size=0.2 1 0.2
Joints:
- added joint BackLeg_Lower: type revolute, parent Back_Leg, child Back_Leg_Lower, origin xyz=0 -1 0 rpy=0 0 0, axis 1 0 0, limit lower=-3.14159 upper=3.14159 effort=0.0 velocity=0.0
- added joint FrontLeg_Lower: type revolute, parent Front_Leg, child Front_Leg_Lower, origin xyz=0 1 0 rpy=0 0 0, axis 1 0 0, limit lower=-3.14159 upper=3.14159 effort=0.0 velocity=0.0
- added joint LeftLeg_Lower: type revolute, parent Left_Leg, child Left_Leg_Lower, origin xyz=1 0 0 rpy=0 0 0, axis 0 1 0, limit lower=-3.14159 upper=3.14159 effort=0.0 velocity=0.0
- added joint RightLeg_Lower: type revolute, parent Right_Leg, child Right_Leg_Lower, origin xyz=-1 0 0 rpy=0 0 0, axis 0 1 0, limit lower=-3.14159 upper=3.14159 effort=0.0 velocity=0.0
- added joint Torso_LeftLeg: type revolute, parent Torso, child Left_Leg, origin xyz=0.5 0 1 rpy=0 0 0, axis 0 1 0, limit lower=-3.14159 upper=3.14159 effort=0.0 velocity=0.0
- added joint Torso_RightLeg: type revolute, parent Torso, child Right_Leg, origin xyz=-0.5 0 1 rpy=0 0 0, axis 0 1 0, limit lower=-3.14159 upper=3.14159 effort=0.0 velocity=0.0
- joint Torso_BackLeg: axis 0 1 0 -> 1 0 0; origin xyz=-0.5 0 1 rpy=0 0 0 -> xyz=0 -0.5 1 rpy=0 0 0
- joint Torso_FrontLeg: axis 0 1 0 -> 1 0 0; origin xyz=0.5 0 1 rpy=0 0 0 -> xyz=0 0.5 1 rpy=0 0 0

Commit message: Created DogQuad Body structure and neurons

File: body.urdf (robot description, URDF)
Before this commit: robot robot, 9 links, 8 joints
Links:
- removed link Back_Leg
- removed link Back_Leg_Lower
- removed link Front_Leg
- removed link Front_Leg_Lower
- removed link Left_Leg
- removed link Left_Leg_Lower
- removed link Right_Leg
- removed link Right_Leg_Lower
- added link Back_Left_Leg, mass 1; collision box size=0.25 0.25 1; visual box size=0.25 0.25 1
- added link Back_Left_Leg_Lower, mass 1; collision box size=1 0.25 0.25; visual box size=1 0.25 0.25
- added link Back_Right_Leg, mass 1; collision box size=0.25 0.25 1; visual box size=0.25 0.25 1
- added link Back_Right_Leg_Lower, mass 1; collision box size=1 0.25 0.25; visual box size=1 0.25 0.25
- added link Front_Left_Leg, mass 1; collision box size=0.25 0.25 1; visual box size=0.25 0.25 1
- added link Front_Left_Leg_Lower, mass 1; collision box size=1 0.25 0.25; visual box size=1 0.25 0.25
- added link Front_Right_Leg, mass 1; collision box size=0.25 0.25 1; visual box size=0.25 0.25 1
- added link Front_Right_Leg_Lower, mass 1; collision box size=1 0.25 0.25; visual box size=1 0.25 0.25
- link Torso: geometry collision box size=3 1 1; visual box size=3 1 1
Joints:
- removed joint BackLeg_Lower
- removed joint FrontLeg_Lower
- removed joint LeftLeg_Lower
- removed joint RightLeg_Lower
- removed joint Torso_BackLeg
- removed joint Torso_FrontLeg
- removed joint Torso_LeftLeg
- removed joint Torso_RightLeg
- added joint Back_Left_To_Lower: type revolute, parent Back_Left_Leg, child Back_Left_Leg_Lower, origin xyz=0 -0.125 -1 rpy=0 0 0, axis 0 1 0, limit lower=-3.14159 upper=3.14159 effort=0.0 velocity=0.0
- added joint Back_Right_To_Lower: type revolute, parent Back_Right_Leg, child Back_Right_Leg_Lower, origin xyz=0 0.125 -1 rpy=0 0 0, axis 0 1 0, limit lower=-3.14159 upper=3.14159 effort=0.0 velocity=0.0
- added joint Front_Left_To_Lower: type revolute, parent Front_Left_Leg, child Front_Left_Leg_Lower, origin xyz=0 -0.125 -1 rpy=0 0 0, axis 0 1 0, limit lower=-3.14159 upper=3.14159 effort=0.0 velocity=0.0
- added joint Front_Right_To_Lower: type revolute, parent Front_Right_Leg, child Front_Right_Leg_Lower, origin xyz=0 0.125 -1 rpy=0 0 0, axis 0 1 0, limit lower=-3.14159 upper=3.14159 effort=0.0 velocity=0.0
- added joint Torso_To_Back_Left: type revolute, parent Torso, child Back_Left_Leg, origin xyz=2.25 -0.5 1 rpy=0 0 0, axis 0 1 0, limit lower=-3.14159 upper=3.14159 effort=0.0 velocity=0.0
- added joint Torso_To_Back_Right: type revolute, parent Torso, child Back_Right_Leg, origin xyz=2.25 0.5 1 rpy=0 0 0, axis 0 1 0, limit lower=-3.14159 upper=3.14159 effort=0.0 velocity=0.0
- added joint Torso_To_Front_Left: type revolute, parent Torso, child Front_Left_Leg, origin xyz=0.125 -0.5 1 rpy=0 0 0, axis 0 1 0, limit lower=-3.14159 upper=3.14159 effort=0.0 velocity=0.0
- added joint Torso_To_Front_Right: type revolute, parent Torso, child Front_Right_Leg, origin xyz=0.125 0.5 1 rpy=0 0 0, axis 0 1 0, limit lower=-3.14159 upper=3.14159 effort=0.0 velocity=0.0

Commit message: Added hidden neurons to the Neural Network, currently 2

File: body.urdf (robot description, URDF)
Before this commit: robot robot, 9 links, 8 joints
Links:
- link Torso: geometry collision box size=3 0.5 0.5; visual box size=3 0.5 0.5
Joints:
- joint Torso_To_Back_Left: origin xyz=2.25 -0.5 1 rpy=0 0 0 -> xyz=2.25 -0.25 1 rpy=0 0 0
- joint Torso_To_Back_Right: origin xyz=2.25 0.5 1 rpy=0 0 0 -> xyz=2.25 0.25 1 rpy=0 0 0
- joint Torso_To_Front_Left: origin xyz=0.125 -0.5 1 rpy=0 0 0 -> xyz=0.125 -0.25 1 rpy=0 0 0
- joint Torso_To_Front_Right: origin xyz=0.125 0.5 1 rpy=0 0 0 -> xyz=0.125 0.25 1 rpy=0 0 0

Commit message: added feet to legs to help with walking

File: body.urdf (robot description, URDF)
Before this commit: robot robot, 9 links, 8 joints
Links:
- added link Back_Left_Foot, mass 1; collision box size=0.35 0.35 0.35; visual box size=0.35 0.35 0.35
- added link Back_Right_Foot, mass 1; collision box size=0.35 0.35 0.35; visual box size=0.35 0.35 0.35
- added link Front_Left_Foot, mass 1; collision box size=0.35 0.35 0.35; visual box size=0.35 0.35 0.35
- added link Front_Right_Foot, mass 1; collision box size=0.35 0.35 0.35; visual box size=0.35 0.35 0.35
Joints:
- added joint Back_Left_Ankle: type revolute, parent Back_Left_Leg_Lower, child Back_Left_Foot, origin xyz=-1.25 -0.2 0 rpy=0 0 0, axis 1 0 0, limit lower=-3.14159 upper=3.14159 effort=0.0 velocity=0.0
- added joint Back_Right_Ankle: type revolute, parent Back_Right_Leg_Lower, child Back_Right_Foot, origin xyz=-1.25 0.2 0 rpy=0 0 0, axis 1 0 0, limit lower=-3.14159 upper=3.14159 effort=0.0 velocity=0.0
- added joint Front_Left_Ankle: type revolute, parent Front_Left_Leg_Lower, child Front_Left_Foot, origin xyz=-1.25 -0.2 0 rpy=0 0 0, axis 1 0 0, limit lower=-3.14159 upper=3.14159 effort=0.0 velocity=0.0
- added joint Front_Right_Ankle: type revolute, parent Front_Right_Leg_Lower, child Front_Right_Foot, origin xyz=-1.25 0.2 0 rpy=0 0 0, axis 1 0 0, limit lower=-3.14159 upper=3.14159 effort=0.0 velocity=0.0
